File: Hardware/Smart Building.kicad_pcb (KiCad board)
At the start: 2 copper layers, 11 parts, among them J2 DHT11, J3 Screw_Terminal_01x03, J4 Screw_Terminal_01x03, J5 Conn_01x06_Pin, J6 ZMPT101b, J7 ACS712, K1 Relay_SPDT, K2 Relay_SPDT, U1 ESP32-DEVKIT-V1

Commit message: memperbarui rangkaian chematic dan board dengan menambahkan sensor tegangan baterai
Parts:
- added J1: Conn_01x02_Pin, Connector_JST:JST_EH_B2B-EH-A_1x02_P2.50mm_Vertical, F.Cu at (131.2, 59.0)
- added R1: R, Resistor_THT:R_Axial_DIN0207_L6.3mm_D2.5mm_P10.16mm_Horizontal, F.Cu at (125.1, 86.2)
- added R2: R, Resistor_THT:R_Axial_DIN0207_L6.3mm_D2.5mm_P10.16mm_Horizontal, F.Cu at (135.2, 89.5)
- added SW1: SW_SPDT, Button_Switch_THT:SW_Slide-03_Wuerth-WS-SLTV_10x2.5x6.4_P2.54mm, F.Cu at (143.2, 59.0)
- J5: value Conn_01x06_Pin -> RTC
Connections:
- U1 pad 21: unconnected-(U1-D32-Pad21) -> Net-(U1-D32)
Routing:
- net +7.5V: track 0.00 -> 28.2 mm, vias 0 -> 1
- net +5V: track 0.00 -> 14.4 mm
- net Net-(U1-D32): track 0.00 -> 12.8 mm
- net Net-(J1-Pin_1): track 0.00 -> 9.46 mm
- net (no net): vias 0 -> 4
