File: Hardware/Smart Building.kicad_pcb (KiCad board)
At the start: 2 copper layers, 11 parts, among them J2 DHT11, J3 Screw_Terminal_01x03, J4 Screw_Terminal_01x03, J5 Conn_01x06_Pin, J6 ZMPT101b, J7 ACS712, K1 Relay_SPDT, K2 Relay_SPDT, U1 ESP32-DEVKIT-V1

Commit message: memperbaiki branch
Other:
- board outline added: 86.7 x 77.9 mm
